File: kicad/rev-a/IphoneFM.kicad_sch (KiCad schematic)
At the start: 16 parts, among them J1 TYPE-C-31-M-12, J2 BWSMA-KWE-Z001, SW1 MSK12C02, SW2 EVQ-P7J01P, SW3 TDP06H1SBD1, U1 STM32U535CEU6, U2 LMX2571NJKR, U3 AP2112K-3.3TRG1, U4 SI4705-D60-GM, U5 PE42421SCAA-Z, U6 USBLC6-2SC6, U7 PE43711B-Z, Y2 OT322520MJBA4SL 20MHz

Commit message: Step 1.16: D1 (LED_RAGB), D3-D4 (TPD1E05U06DPY), D5 (D_TVS) placed
Co-Authored-By: Claude Opus 5.5 <noreply@anthropic.com>
Parts:
- added D1: XL-1615RGBC-RF, symbol Device:LED_RAGB
- added D3, D4: TPD1E05U06DPYR, Package_SON:Texas_DPY0002A_0.6x1mm_P0.65mm, symbol Power_Protection:TPD1E05U06DPY
- added D5: RCLAMP0521PATCT, symbol Device:D_TVS
Changed lines of the file:
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@@
+		)
+	)
+	(symbol
+		(lib_id "Device:LED_RAGB")
+		(at 142.24 302.26 0)
+		(unit 1)
+		(exclude_from_sim no)
+		(in_bom yes)
+		(on_board yes)
+		(dnp no)
+		(property "Reference" "D1"
+			(at 142.24 298.45 0)
+			(effects (font (size 1.27 1.27)))
+		)
+		(property "Value" "XL-1615RGBC-RF"
+			(at 142.24 306.07 0)
+			(effects (font (size 1.27 1.27)))
+		)
+		(property "Footprint" ""
+			(at 142.24 302.26 0)
+			(effects (font (size 1.27 1.27)) (hide yes))
+		)
+		(property "Datasheet" "~"
+			(at 142.24 302.26 0)
+			(effects (font (size 1.27 1.27)) (hide yes))
+		)
+		(instances
+			(project "IphoneFM"
+				(path "/efee88c9-028d-4fdb-86e0-0a4145b330e1"
+					(reference "D1") (unit 1)
+				)
+			)
+		)
+	)
+	(symbol
+		(lib_id "Power_Protection:TPD1E05U06DPY")
+		(at 60.96 124.46 0)
+		(unit 1)
+		(exclude_from_sim no)
+		(in_bom yes)
+		(on_board yes)
+		(dnp no)
+		(property "Reference" "D3"
+			(at 60.96 120.65 0)
+			(effects (font (size 1.27 1.27)))
+		)
+		(property "Value" "TPD1E05U06DPYR"
+			(at 60.96 128.27 0)
+			(effects (font (size 1.27 1.27)))
+		)
+		(property "Footprint" "Package_SON:Texas_DPY0002A_0.6x1mm_P0.65mm"
+			(at 60.96 124.46 0)
+			(effects (font (size 1.27 1.27)) (hide yes))
+		)
+		(property "Datasheet" "~"
+			(at 60.96 124.46 0)
+			(effects (font (size 1.27 1.27)) (hide yes))
+		)
+		(instances
+			(project "IphoneFM"
+				(path "/efee88c9-028d-4fdb-86e0-0a4145b330e1"
+					(reference "D3") (unit 1)
+				)
+			)
+		)
+	)
+	(symbol
+		(lib_id "Power_Protection:TPD1E05U06DPY")
+		(at 76.2 124.46 0)
+		(unit 1)
+		(exclude_from_sim no)
+		(in_bom yes)
+		(on_board yes)
+		(dnp no)
+		(property "Reference" "D4"
+			(at 76.2 120.65 0)
+			(effects (font (size 1.27 1.27)))
+		)
+		(property "Value" "TPD1E05U06DPYR"
+			(at 76.2 128.27 0)
+			(effects (font (size 1.27 1.27)))
+		)
+		(property "Footprint" "Package_SON:Texas_DPY0002A_0.6x1mm_P0.65mm"
+			(at 76.2 124.46 0)
+			(effects (font (size 1.27 1.27)) (hide yes))
+		)
+		(property "Datasheet" "~"
+			(at 76.2 124.46 0)
+			(effects (font (size 1.27 1.27)) (hide yes))
+		)
+		(instances
+			(project "IphoneFM"
+				(path "/efee88c9-028d-4fdb-86e0-0a4145b330e1"
+					(reference "D4") (unit 1)
+				)
+			)
+		)
+	)
+	(symbol
+		(lib_id "Device:D_TVS")
+		(at 551.18 177.8 90)
+		(unit 1)
+		(exclude_from_sim no)
+		(in_bom yes)
+		(on_board yes)
+		(dnp no)
+		(property "Reference" "D5"
+			(at 551.18 173.99 90)
+			(effects (font (size 1.27 1.27)))
+		)
+		(property "Value" "RCLAMP0521PATCT"
+			(at 551.18 181.61 90)
+			(effects (font (size 1.27 1.27)))
+		)
+		(property "Footprint" ""
+			(at 551.18 177.8 90)
+			(effects (font (size 1.27 1.27)) (hide yes))
+		)
+		(property "Datasheet" "~"
+			(at 551.18 177.8 0)
+			(effects (font (size 1.27 1.27)) (hide yes))
+		)
+		(instances
+			(project "IphoneFM"
+				(path "/efee88c9-028d-4fdb-86e0-0a4145b330e1"
+					(reference "D5") (unit 1)
+				)
+			)
 		)
 	)

Commit message: Step 1.17: all 74 passives placed beside their pins (tools/sch_place.py)
Also fixes the symbol-replace bug in kicad_symbol.py that left stale copies of
OT322520MJBA4SL and RK10J11R0A0H in the library; the sheet now carries the
rebuilt wheel symbol (lands on the left) and matches the library.

Co-Authored-By: Claude Opus 5.5 <noreply@anthropic.com>
Parts:
- added C1, C2, C27, C8: 1 µF X7R 16 V, Capacitor_SMD:C_0603_1608Metric, symbol Device:C
- added C10, C11, C13, C14, C15, C16, C17, C18, C19, C20, C21, C22, C33, C39, C4, C40, C41, C5, C6, C7: 100 nF X7R 16 V, Capacitor_SMD:C_0402_1005Metric, symbol Device:C
- added C12, C3: 10 µF X5R 16 V, Capacitor_SMD:C_0805_2012Metric, symbol Device:C
- added C23: 2.2 µF X5R 16 V, Capacitor_SMD:C_0603_1608Metric, symbol Device:C
- added C24, C26: 100 pF C0G, Capacitor_SMD:C_0402_1005Metric, symbol Device:C
- added C25: 1.5 nF C0G, Capacitor_SMD:C_0402_1005Metric, symbol Device:C
- added C28, C30, C37, C38: 33 pF C0G, Capacitor_SMD:C_0402_1005Metric, symbol Device:C
- added C29: 56 pF C0G, Capacitor_SMD:C_0402_1005Metric, symbol Device:C
- added C31, C34: 1 nF C0G, Capacitor_SMD:C_0402_1005Metric, symbol Device:C
- added C32: 22 nF X7R 50 V, Capacitor_SMD:C_0402_1005Metric, symbol Device:C
- added C35: 6 pF C0G, Capacitor_SMD:C_0402_1005Metric, symbol Device:C
- added C36: 3.3 pF C0G, Capacitor_SMD:C_0402_1005Metric, symbol Device:C
- added C9: 4.7 µF X7R 16 V, Capacitor_SMD:C_0805_2012Metric, symbol Device:C
- added FB1: 75 Ω at 100 MHz, Inductor_SMD:L_0402_1005Metric, symbol Device:FerriteBead
- added FB2, FB3: 600 Ω at 100 MHz, Inductor_SMD:L_0402_1005Metric, symbol Device:FerriteBead
- added L1: 150 nH 2%, Inductor_SMD:L_0603_1608Metric, symbol Device:L
- added L2, L3: 100 nH 2%, Inductor_SMD:L_0603_1608Metric, symbol Device:L
- added R1, R2: 5.1 kΩ 1%, Resistor_SMD:R_0402_1005Metric, symbol Device:R
- added R10, R11, R12, R13, R14, R15, R19, R3, R9: 10 kΩ 1%, Resistor_SMD:R_0402_1005Metric, symbol Device:R
- added R16, R17: 1 kΩ 1%, Resistor_SMD:R_0402_1005Metric, symbol Device:R
- added R18: 100 kΩ 1%, Resistor_SMD:R_0402_1005Metric, symbol Device:R
- added R20, R21: 6.8 kΩ 1%, Resistor_SMD:R_0402_1005Metric, symbol Device:R
- added R22: 604 Ω 1%, Resistor_SMD:R_0402_1005Metric, symbol Device:R
- added R23, R24: 2 kΩ 1%, Resistor_SMD:R_0402_1005Metric, symbol Device:R
- added R25: 510 Ω 1%, Resistor_SMD:R_0402_1005Metric, symbol Device:R
- added R26, R27: 390 Ω 1%, Resistor_SMD:R_0402_1005Metric, symbol Device:R
- added R4, R6, R7, R8: 33 Ω 1%, Resistor_SMD:R_0402_1005Metric, symbol Device:R
- added R5: 1.1 kΩ 1%, Resistor_SMD:R_0402_1005Metric, symbol Device:R
Other:
- moved on the sheet: RV1, RV2, RV3

Commit message: Step 1.17 ticked; step 1.18: value, MPN, LCSC and manufacturer on all 94 symbols from netlist.json (tools/sch_fields.py)
Co-Authored-By: Claude Opus 5.5 <noreply@anthropic.com>
Parts:
- C1, C2, C27, C8: LCSC (none) -> C59782; MPN (none) -> CL10B105KO8NNNC; Manufacturer (none) -> Samsung
- C10, C11, C13, C14, C15, C16, C17, C18, C19, C20, C21, C22, C33, C39, C4, C40, C41, C5, C6, C7: LCSC (none) -> C1525; MPN (none) -> CL05B104KO5NNNC; Manufacturer (none) -> Samsung
- C12, C3: LCSC (none) -> C1713; MPN (none) -> CL21A106KOQNNNE; Manufacturer (none) -> Samsung
- C23: LCSC (none) -> C23630; MPN (none) -> CL10A225KO8NNNC; Manufacturer (none) -> Samsung
- C24, C26: LCSC (none) -> C26409; MPN (none) -> CL05C101JB5NNNC; Manufacturer (none) -> Samsung
- C25: LCSC (none) -> C668348; MPN (none) -> GRM1555C1H152JA01D; Manufacturer (none) -> Murata
- C28, C30, C37, C38: LCSC (none) -> C70465; MPN (none) -> CL05C330JB5NNNC; Manufacturer (none) -> Samsung
- C29: LCSC (none) -> C107007; MPN (none) -> CC0402JRNPO9BN560; Manufacturer (none) -> Yageo
- C31, C34: LCSC (none) -> C76947; MPN (none) -> GRM1555C1H102JA01D; Manufacturer (none) -> Murata
- C32: LCSC (none) -> C77023; MPN (none) -> GRM155R71H223KA12D; Manufacturer (none) -> Murata
- C35: LCSC (none) -> C161330; MPN (none) -> GJM1555C1H6R0CB01D; Manufacturer (none) -> Murata
- C36: LCSC (none) -> C76968; MPN (none) -> GRM1555C1H3R3CA01D; Manufacturer (none) -> Murata
- C9: LCSC (none) -> C408144; MPN (none) -> GRM21BR71C475KE51L; Manufacturer (none) -> Murata
- D1: value XL-1615RGBC-RF -> RGB LED, common anode; LCSC (none) -> C965840; MPN (none) -> XL-1615RGBC-RF; Manufacturer (none) -> XINGLIGHT
- D3, D4: value TPD1E05U06DPYR -> ESD 5.5 V; LCSC (none) -> C436349; MPN (none) -> TPD1E05U06DPYR; Manufacturer (none) -> TI
- D5: value RCLAMP0521PATCT -> ESD 5 V, 0.5 pF; LCSC (none) -> C117554; MPN (none) -> RCLAMP0521PATCT; Manufacturer (none) -> Semtech
- FB1: LCSC (none) -> C113009; MPN (none) -> BLM15GA750SN1D; Manufacturer (none) -> Murata
- FB2, FB3: LCSC (none) -> C76884; MPN (none) -> BLM15AG601SN1D; Manufacturer (none) -> Murata
- J1: value TYPE-C-31-M-12 -> USB 2.0 Type-C; LCSC (none) -> C165948; MPN (none) -> TYPE-C-31-M-12; Manufacturer (none) -> Korean Hroparts
- J2: value BWSMA-KWE-Z001 -> SMA jack; LCSC (none) -> C496551; MPN (none) -> BWSMA-KWE-Z001; Manufacturer (none) -> BAT Wireless
- L1: LCSC (none) -> C113131; MPN (none) -> LQW18ANR15G00D; Manufacturer (none) -> Murata
- L2, L3: LCSC (none) -> C98088; MPN (none) -> LQW18ANR10G00D; Manufacturer (none) -> Murata
- R1, R2: LCSC (none) -> C105872; MPN (none) -> RC0402FR-075K1L; Manufacturer (none) -> Yageo
- R10, R11, R12, R13, R14, R15, R19, R3, R9: LCSC (none) -> C60490; MPN (none) -> RC0402FR-0710KL; Manufacturer (none) -> Yageo
- R16, R17: LCSC (none) -> C106235; MPN (none) -> RC0402FR-071KL; Manufacturer (none) -> Yageo
- R18: LCSC (none) -> C60491; MPN (none) -> RC0402FR-07100KL; Manufacturer (none) -> Yageo
- R20, R21: LCSC (none) -> C93940; MPN (none) -> RC0402FR-076K8L; Manufacturer (none) -> Yageo
- R22: LCSC (none) -> C273693; MPN (none) -> RC0402FR-07604RL; Manufacturer (none) -> Yageo
- R23, R24: LCSC (none) -> C413086; MPN (none) -> ERJ-2RKF2001X; Manufacturer (none) -> Panasonic
- R25: LCSC (none) -> C276273; MPN (none) -> RC0402FR-07510RL; Manufacturer (none) -> Yageo
- R26, R27: LCSC (none) -> C137997; MPN (none) -> RC0402FR-07390RL; Manufacturer (none) -> Yageo
- R4, R6, R7, R8: LCSC (none) -> C138002; MPN (none) -> RC0402FR-0733RL; Manufacturer (none) -> Yageo
- R5: LCSC (none) -> C409028; MPN (none) -> ERJ-2RKF1101X; Manufacturer (none) -> Panasonic
- RV1, RV2, RV3: value RK10J11R0A0H -> 10 kΩ 3B; LCSC (none) -> C470766; MPN (none) -> RK10J11R0A0H; Manufacturer (none) -> Alps
- SW1: value MSK12C02 -> SPDT; LCSC (none) -> C431540; MPN (none) -> MSK12C02; Manufacturer (none) -> Shou Han
- SW2: value EVQ-P7J01P -> SPST; LCSC (none) -> C2828254; MPN (none) -> EVQ-P7J01P; Manufacturer (none) -> Panasonic
- SW3: value TDP06H1SBD1 -> 6 × SPST; LCSC (none) -> C221994; MPN (none) -> TDP06H1SBD1; Manufacturer (none) -> C&K
- U1: value STM32U535CEU6 -> MCU; LCSC (none) -> C22454224; MPN (none) -> STM32U535CEU6; Manufacturer (none) -> ST
- U2: value LMX2571NJKR -> Synthesizer; LCSC (none) -> C440388; MPN (none) -> LMX2571NJKR; Manufacturer (none) -> TI
- U3: value AP2112K-3.3TRG1 -> 3.3 V 600 mA LDO; LCSC (none) -> C51118; MPN (none) -> AP2112K-3.3TRG1; Manufacturer (none) -> Diodes
- U4: value SI4705-D60-GM -> FM receiver; LCSC (none) -> C1526114; MPN (none) -> SI4705-D60-GM; Manufacturer (none) -> Skyworks
- U5: value PE42421SCAA-Z -> SPDT RF switch; LCSC (none) -> C470893; MPN (none) -> PE42421SCAA-Z; Manufacturer (none) -> pSemi
- U6: value USBLC6-2SC6 -> USB ESD array; LCSC (none) -> C7519; MPN (none) -> USBLC6-2SC6; Manufacturer (none) -> ST
- U7: value PE43711B-Z -> Digital step attenuator; LCSC (none) -> C470929; MPN (none) -> PE43711B-Z; Manufacturer (none) -> pSemi
- Y2: value OT322520MJBA4SL 20MHz -> 20 MHz CMOS XO; LCSC (none) -> C725987; MPN (none) -> OT322520MJBA4SL; Manufacturer (none) -> YXC

Commit message: Step 1.18 ticked; step 1.19: power symbols on every VBUS, 3V3, VDDA, RX_VDD and GND pin (tools/sch_power.py)
Passives are turned so ground sits at the bottom and supplies on top, and the
placer now leaves room for the power symbols.

Co-Authored-By: Claude Opus 5.5 <noreply@anthropic.com>
Connections:
- net GND: now reaches D4.2 (GND)
- net GND: now also C1.2, C10.2, C11.2, C12.2, C13.2, C14.2, C15.2, C16.2, C17.2, C18.2, C19.2, C2.2, C20.2, C21.2, C22.2, C23.2, C24.2, C25.2, C27.2, C28.2, C29.2, C3.2, C30.2, C31.2, C32.2, C33.2, C35.2, C36.2, C37.2, C38.2, C39.2, C4.2, C40.2, C41.2, C5.2, C6.2, C7.2, C8.2, C9.2, D3.2 (GND), D5.2 (A2), J1.A1 (GND), J1.A12 (GND), J1.B1 (GND), J1.B12 (GND), J1.SH (SHIELD), J2.2 (Ext), L1.2, R1.2, R10.2, R11.2, R12.2, R13.2, R14.2, R15.2, R18.2, R19.2, R2.2, R3.2, R9.2, RV1.3 (CCW end), RV1.D1 (Dummy), RV1.D2 (Dummy), RV1.M1 (Mounting), RV1.M2 (Mounting), RV2.3 (CCW end), RV2.D1 (Dummy), RV2.D2 (Dummy), RV2.M1 (Mounting), RV2.M2 (Mounting), RV3.3 (CCW end), RV3.D1 (Dummy), RV3.D2 (Dummy), RV3.M1 (Mounting), RV3.M2 (Mounting), SW1.3 (Throw (RX)), SW1.4 (Tab), U1.23 (VSS), U1.35 (VSS), U1.47 (VSS), U1.49 (VSS), U1.8 (VSSA), U2.18 (TrCtl), U2.23 (GND), U2.31 (GND), U2.35 (GND), U2.37 (DAP), U2.5 (FSK_D2), U3.2 (GND), U4.12 (GND), U4.13 (ROUT), U4.14 (LOUT), U4.21 (EP), U4.3 (RFGND), U4.4 (LPI), U4.6 (SENB), U5.2 (GND), U6.2 (GND), U7.1 (C0.25), U7.10 (GND), U7.11 (GND), U7.12 (GND), U7.13 (GND), U7.15 (GND), U7.17 (CLK), U7.18 (SI), U7.25 (EP), U7.3 (P/S), U7.4 (GND), U7.6 (GND), U7.7 (GND), U7.8 (GND), U7.9 (GND), Y2.2 (GND)
- net 3V3: now reaches SW2.1
- net 3V3: now also C11.1, C12.1, C13.1, C14.1, C15.1, C16.1, C17.1, C18.1, C19.1, C2.1, C27.1, C3.1, C4.1, C5.1, C6.1, FB2.1, FB3.1, R16.1, R20.2, R21.2, RV1.1 (CW end), RV2.1 (CW end), RV3.1 (CW end), SW1.1 (Throw (TX)), SW3.10, SW3.11, SW3.12, SW3.7, SW3.8, SW3.9, U1.1 (VBAT), U1.24 (VDD), U1.36 (VDD), U1.48 (VDD), U2.1 (Vcc3p3), U2.15 (VccIO), U2.20 (Vcc3p3), U2.27 (Vcc3p3), U2.32 (VcpExt), U2.33 (VccIO), U2.9 (Vcc3p3), U3.5 (VOUT), U7.16 (LE), U7.2 (VDD), Y2.1 (Tri-state), Y2.4 (VDD)
- net RX_VDD: now reaches U4.10 (VD)
- net RX_VDD: now also C32.1, C33.1, FB3.2, U4.11 (VA)
- net VBUS: now reaches U6.5 (VBUS)
- net VBUS: now also C1.1, D1.2 (A), J1.A4 (VBUS), J1.A9 (VBUS), J1.B4 (VBUS), J1.B9 (VBUS), U3.1 (VIN), U3.3 (EN)
- net VDDA: now reaches U1.9 (VDDA)
- net VDDA: now also C7.1, C8.1, FB2.2
