File: kicad/rev-a/panel/IphoneFM-panel.kicad_pcb (KiCad board)
At the start: 2 copper layers, 78.4 x 90.4 mm, 134 parts, among them J1 USB 2.0 Type-C, J2 SMA jack, SW1 SPDT, SW2 SPST, SW3 6 × SPST, U1 MCU, U2 Synthesizer, U3 3.3 V 600 mA LDO, U4 FM receiver, U5 SPDT RF switch, U6 USB ESD array, U7 Digital step attenuator, Y2 20 MHz CMOS XO

Commit message: JLC Basic-library parts for 14 passive types (same values and sizes, equal or higher ratings; datasheets saved); netlist, schematic, board, notes and wiring page updated
Co-Authored-By: Claude Opus 5.5 <noreply@anthropic.com>
Parts:
- C1, C2, C27, C8: value 1 µF X7R 16 V -> 1 µF X5R 50 V
- C12, C3: value 10 µF X5R 16 V -> 10 µF X5R 25 V
- C31, C34: value 1 nF C0G -> 1 nF X7R 50 V
- C9: value 4.7 µF X7R 16 V -> 4.7 µF X5R 25 V
